Commit message: add bcr_bot

File: description/bcr_bot/bcr_bot.xacro (robot description, xacro)
@@ -20,9 +20,9 @@
     <xacro:property name="traction_track_width" value="0.6"/>
     <xacro:property name="two_d_lidar_update_rate" value="30"/>
-    <xacro:property name="two_d_lidar_sample_size" value="361"/>
+    <xacro:property name="two_d_lidar_sample_size" value="2117"/>
     <xacro:property name="two_d_lidar_min_angle" value="0"/>
     <xacro:property name="two_d_lidar_max_angle" value="360"/>
-    <xacro:property name="two_d_lidar_min_range" value="0.55"/>
-    <xacro:property name="two_d_lidar_max_range" value="16"/>
+    <xacro:property name="two_d_lidar_min_range" value="0.8"/>
+    <xacro:property name="two_d_lidar_max_range" value="40"/>
     <xacro:property name="camera_baseline" value="0.06"/>
     <xacro:property name="camera_height" value="0.10"/>

Commit message: rix gz parmas

File: description/bcr_bot/bcr_bot.xacro (robot description, xacro)
@@ -19,5 +19,5 @@
     <xacro:property name="traction_wheel_width" value="0.05"/>
     <xacro:property name="traction_track_width" value="0.6"/>
-    <xacro:property name="two_d_lidar_update_rate" value="30"/>
+    <xacro:property name="two_d_lidar_update_rate" value="20"/>
     <xacro:property name="two_d_lidar_sample_size" value="2117"/>
     <xacro:property name="two_d_lidar_min_angle" value="0"/>

File: description/bcr_bot/gz.xacro (robot description, xacro)
@@ -36,5 +36,5 @@
             <tf_topic>/tf</tf_topic>
             <dimensions>2</dimensions>
-            <odom_publish_frequency>10</odom_publish_frequency>
+            <odom_publish_frequency>30</odom_publish_frequency>
         </plugin>
     </gazebo>
