Commit message: update ammr sj xacro

File: description/ammr_sj/ammr_sj.xacro (robot description, xacro)
@@ -1,235 +1,232 @@
-<?xml version="1.0" ?>
-<robot name="ammr_sj" xmlns:xacro="http://www.ros.org/wiki/xacro">
-    <!-- CONSTANTS -->
-    <!-- Math -->
-    <xacro:property name="PI" value="3.1415926535897931"/>
-    <!-- ARGUMENTS -->
-    <xacro:property name="pkg_path" value="$(find amr_sim)"/>
-    <xacro:property name="urdf_dir" value="${pkg_path}/description/hamr"/>
-    <xacro:arg name="is_simulation" default="false" />
-    <xacro:arg name="use_fake_hardware" default="true" />
-    <xacro:arg name="fake_sensor_commands" default="false" />
-    <xacro:property name="param_file" value="${pkg_path}/param/ammr_sj/amr_swerve_controller.yaml"/>
-    <!-- Chassis dimensions -->
-    <xacro:property name="chassis_mass" value="1.0" /> <!-- arbitrary value for base mass -->
-    <xacro:property name="chassis_length" value="1.0" />
-    <xacro:property name="chassis_width" value="0.5" />
-    <xacro:property name="chassis_height" value="0.4" />
-    <!-- Suspension dimensions -->
-    <xacro:property name="wheel_offset" value="0.01" />
-    <xacro:property name="steering_mass" value="0.2" />
-    <xacro:property name="steering_radius" value="0.15" />
-    <xacro:property name="steering_thickness" value="0.01" />
-    <xacro:property name="scan_height" value="0.0995" /> <!-- 99.5mm -->
-    <!-- Wheel dimensions -->
-    <xacro:property name="wheel_mass" value="0.2" />
-    <xacro:property name="wheel_radius" value="0.075" /> <!-- 75mm -->
-    <xacro:property name="wheel_width" value="0.05" /> <!-- 50mm -->
-    <xacro:property name="wheel_base" value="0.728" /> <!-- 728mm -->
-    <xacro:property name="wheel_track" value="0.274" /> <!-- 274mm -->
-    <!-- Caster wheel dimensions -->
-    <xacro:property name="caster_mass" value="0.1" />
-    <xacro:property name="caster_radius" value="0.05" />
-    <xacro:property name="caster_width" value="0.03" />
-    <!-- -->
-    <xacro:property name="front_x_reflect" value="1" />
-    <xacro:property name="rear_x_reflect" value="-1" />
-    <xacro:property name="left_y_reflect" value="1" />
-    <xacro:property name="right_y_reflect" value="-1" />
-    <!-- INCLUDES -->
-    <xacro:include filename="materials.xacro" />
-    <xacro:include filename="ammr_sj_macros.xacro" />
-    <xacro:include filename="ammr_sj_gazebo.xacro" />
-    <!-- MODEL -->
-    <!--
-      An empty base footprint that describes the origin of the robot on the ground
-    -->
-    <link name="base_footprint">
-    </link>
-    <!--
-      base_link: The center of gravity (CoG) of the chassis
-      Joint from base_footprint (ground) to base_link (at chassis CoG height)
-    -->
-    <joint name="joint_base_to_footprint" type="fixed">
-        <!-- base_link is positioned at the center of the chassis (CoG) -->
-        <origin rpy="0 0 0" xyz="0 0 ${wheel_radius}"/>
-        <parent link="base_footprint"/>
-        <child link="base_link"/>
-    </joint>
-    <link name="base_link">
-        <!-- Chassis inertial properties at the CoG -->
-        <inertial>
-            <origin rpy="0 0 0" xyz="0 0 0"/>
-            <mass value="${chassis_mass}"/>
-            <inertia
-                ixx="${chassis_mass / 12.0 * (chassis_width * chassis_width + chassis_height * chassis_height)}"
-                ixy="0"
-                ixz="0"
-                iyy="${chassis_mass / 12.0 * (chassis_length * chassis_length + chassis_height * chassis_height)}"
-                iyz="0"
-                izz="${chassis_mass / 12.0 * (chassis_length * chassis_length + chassis_width * chassis_width)}"/>
-        </inertial>
-        <!-- Chassis visual representation -->
-        <visual>
-            <origin rpy="0 0 0" xyz="0 0 0"/>
-            <geometry>
-                <box size="${chassis_length} ${chassis_width} ${chassis_height}" />
-            </geometry>
-            <material name="orange"/>
-        </visual>
-        <!-- Chassis collision geometry -->
-        <collision>
-            <origin rpy="0 0 0" xyz="0 0 0"/>
-            <geometry>
-                <box size="${chassis_length} ${chassis_width} ${chassis_height}" />
-            </geometry>
-        </collision>
-    </link>
-    <!--
-        Right front wheel assembly (motorized)
-    -->
-    <xacro:drive_module_assembly
-        name="right_front"
-        chassis_length="${chassis_length}"
-        chassis_width="${chassis_width}"
-        chassis_height="${chassis_height}"
-        wheel_mass="${wheel_mass}"
-        wheel_radius="${wheel_radius}"
-        wheel_width="${wheel_width}"
-        wheel_base="${wheel_base}"
-        wheel_track="${wheel_track}"
-        steering_mass="${steering_mass}"
-        steering_radius="${steering_radius}"
-        steering_thickness="${steering_thickness}"
-        offset="${wheel_offset}"
-        x_reflect="${front_x_reflect}"
-        y_reflect="${right_y_reflect}" />
-    <!--
-        Left rear wheel assembly (motorized)
-    -->
-    <xacro:drive_module_assembly
-        name="left_rear"
-        chassis_length="${chassis_length}"
-        chassis_width="${chassis_width}"
-        chassis_height="${chassis_height}"
-        wheel_mass="${wheel_mass}"
-        wheel_radius="${wheel_radius}"
-        wheel_width="${wheel_width}"
-        wheel_base="${wheel_base}"
-        wheel_track="${wheel_track}"
-        steering_mass="${steering_mass}"
-        steering_radius="${steering_radius}"
-        steering_thickness="${steering_thickness}"
-        offset="${wheel_offset}"
-        x_reflect="${rear_x_reflect}"
-        y_reflect="${left_y_reflect}" />
-    <!--
-        Left front caster wheel (passive)
-    -->
-    <xacro:caster_wheel_assembly
-        name="left_front"
-        mass="${caster_mass}"
-        radius="${caster_radius}"
-        width="${caster_width}"
-        x_pos="${front_x_reflect * (0.5 * wheel_base)}"
-        y_pos="${left_y_reflect * (0.5 * wheel_track)}" />
-    <!--
-        Right rear caster wheel (passive)
-    -->
-    <xacro:caster_wheel_assembly
-        name="right_rear"
-        mass="${caster_mass}"
-        radius="${caster_radius}"
-        width="${caster_width}"
-        x_pos="${rear_x_reflect * (0.5 * wheel_base)}"
-        y_pos="${right_y_reflect * (0.5 * wheel_track)}" />
-    <ros2_control name="AmmrSjJointControl" type="system">
-        <xacro:if value="$(arg is_simulation)">
-            <hardware>
-                <plugin>gz_ros2_control/GazeboSimSystem</plugin>
-            </hardware>
-        </xacro:if>
-        <xacro:unless value="$(arg is_simulation)">
-            <xacro:if value="$(arg use_fake_hardware)">
-                <hardware>
-                    <plugin>mock_components/GenericSystem</plugin>
-                </hardware>
-            </xacro:if>
-            <xacro:unless value="$(arg use_fake_hardware)">
-                <!-- USE REAL HARDWARE HERE -->
-                <hardware>
-                </hardware>
-            </xacro:unless>
-        </xacro:unless>
-        <xacro:steering_module_controller name="right_front" />
-        <xacro:steering_module_controller name="left_rear" />
-    </ros2_control>
-    <!-- Sensors -->
-    <!-- IMU -->
-    <xacro:imu_frame name="imu_frame" parent_link="base_link">
-        <origin rpy="0 0 0" xyz="0.0 0.0 0.0"/>
-    </xacro:imu_frame>
-    <joint name="base_link_to_base_scan" type="fixed">
-        <parent link="base_link"/>
-        <child link="base_scan"/>
-        <origin xyz="0.0 0.0 ${scan_height - wheel_radius}"/>
-    </joint>
-    <link name="base_scan">
-    </link>
-    <!-- LIDAR Front (left front) -->
-    <joint name="base_scan_to_lidar_front" type="fixed">
-        <parent link="base_scan"/>
-        <child link="lidar_front"/>
-        <origin xyz="0.551175 0.324045 0.0" rpy="3.14159 0 0.7854"/>
-    </joint>
-    <link name="lidar_front">
-        <visual>
-            <origin rpy="0 0 0" xyz="0 0 0"/>
-            <geometry>
-                <cylinder radius="0.03" length="0.082"/>
-            </geometry>
-            <material name="Red"/>
-        </visual>
-        <collision>
-            <origin rpy="0 0 0" xyz="0 0 0"/>
-            <geometry>
-                <cylinder radius="0.03" length="0.082"/>
-            </geometry>
-        </collision>
-        <inertial>
-            <mass value="1.0"/>
-            <origin xyz="0 0 0" rpy="0 0 0"/>
-            <inertia ixx="0.00146" ixy="0" ixz="0" iyy="0.00146" iyz="0" izz="0.00125"/>
-        </inertial>
-    </link>
-    <!-- LIDAR Back (right rear) -->
-    <joint name="base_scan_to_lidar_back" type="fixed">
-        <parent link="base_scan"/>
-        <child link="lidar_back"/>
-        <origin xyz="-0.551175 -0.324045 0.0" rpy="3.14159 0 -2.35619"/>
-    </joint>
-    <link name="lidar_back">
-        <visual>
-            <origin rpy="0 0 0" xyz="0 0 0"/>
-            <geometry>
-                <cylinder radius="0.03" length="0.082"/>
-            </geometry>
-            <material name="Red"/>
-        </visual>
-        <collision>
-            <origin rpy="0 0 0" xyz="0 0 0"/>
-            <geometry>
-                <cylinder radius="0.03" length="0.082"/>
-            </geometry>
-        </collision>
-        <inertial>
-            <mass value="1.0"/>
-            <origin xyz="0 0 0" rpy="0 0 0"/>
-            <inertia ixx="0.00146" ixy="0" ixz="0" iyy="0.00146" iyz="0" izz="0.00125"/>
-        </inertial>
-    </link>
-    <!-- Bump -->
-    <!-- Sonar -->
-    <!-- IR -->
-    <!-- Cliff sensors -->
+<?xml version="1.0"?>
+<robot name="hamr" xmlns:xacro="http://www.ros.org/wiki/xacro">
+  <!-- =========================================================
+       PACKAGE PATHS
+       ========================================================= -->
+  <xacro:property name="pkg_path" value="$(find amr_sim)"/>
+  <xacro:property name="urdf_dir" value="${pkg_path}/description/ammr_sj"/>
+  <xacro:property name="param_file" value="${pkg_path}/param/ammr_sj/amr_swerve_control.yaml"/>
+  <!-- Math -->
+  <xacro:property name="PI" value="3.1415926535897931"/>
+  <!-- ARGUMENTS -->
+  <xacro:arg name="chassis_version" default="v1"/>
+  <!-- Chassis dimensions -->
+  <xacro:property name="chassis_mass" value="1.0"/>
+  <xacro:property name="chassis_length" value="1.244"/>
+  <xacro:property name="chassis_width"  value="0.794"/>
+  <xacro:property name="chassis_height" value="0.692"/>
+  <xacro:property name="chassis_bottom_z" value="0.028"/>
+  <!-- Suspension dimensions -->
+  <xacro:property name="wheel_offset" value="0.01"/>
+  <xacro:property name="steering_mass" value="0.2"/>
+  <xacro:property name="steering_radius" value="0.05"/>
+  <xacro:property name="steering_thickness" value="0.01"/>
+  <!-- Wheel dimensions -->
+  <xacro:property name="wheel_mass" value="0.2"/>
+  <xacro:property name="wheel_radius" value="0.15"/>
+  <xacro:property name="wheel_width" value="0.04"/>
+  <xacro:property name="wheel_base" value="0.728"/>
+  <xacro:property name="wheel_track" value="0.274"/>
+  <xacro:property name="scan_height" value="0.0995"/>
+  <xacro:property name="front_x_reflect" value="1"/>
+  <xacro:property name="rear_x_reflect"  value="-1"/>
+  <xacro:property name="left_y_reflect"  value="1"/>
+  <xacro:property name="right_y_reflect" value="-1"/>
+  <xacro:property name="caster_trail" value="0.01"/>
+  <!-- INCLUDES -->
+  <xacro:include filename="${urdf_dir}/materials.xacro"/>
+  <xacro:include filename="${urdf_dir}/ammr_sj_macros.xacro"/>
+  <xacro:include filename="${urdf_dir}/ammr_sj_gazebo.xacro"/>
+  <!-- =========================================================
+       1) BASE FRAMES
+       ========================================================= -->
+  <link name="base_footprint"/>
+  <link name="base_link">
+    <inertial>
+      <origin xyz="0 0 0.0" rpy="0 0 0"/>
+      <mass value="${chassis_mass}"/>
+      <inertia
+        ixx="${chassis_mass / 12.0 * (chassis_width  * chassis_width  + chassis_height * chassis_height)}"
+        ixy="0" ixz="0"
+        iyy="${chassis_mass / 12.0 * (chassis_length * chassis_length + chassis_height * chassis_height)}"
+        iyz="0"
+        izz="${chassis_mass / 12.0 * (chassis_length * chassis_length + chassis_width  * chassis_width)}"/>
+    </inertial>
+  </link>
+  <joint name="joint_base_to_footprint" type="fixed">
+    <parent link="base_footprint"/>
+    <child  link="base_link"/>
+    <origin xyz="0 0 ${chassis_bottom_z + 0.5 * chassis_height}" rpy="0 0 0"/>
+  </joint>
+  <!-- =========================================================
+       2) CHASSIS LINK (mounting / body reference)
+       ========================================================= -->
+  <link name="chassis_link">
+    <visual>
+      <origin xyz="0 0 0.0" rpy="0 0 0"/>
+    </visual>
+    <collision>
+      <origin xyz="0 0 0.0" rpy="0 0 0"/>
+    </collision>
+  </link>
+  <joint name="base_to_chassis" type="fixed">
+    <parent link="base_link"/>
+    <child  link="chassis_link"/>
+    <origin xyz="0 0 0" rpy="0 0 0"/>
+  </joint>
+  <!-- =========================================================
+       3) DRIVE MODULES / CASTERS
+       ========================================================= -->
+  <xacro:drive_module_assembly
+    name="right_front"
+    chassis_length="${chassis_length}"
+    chassis_width="${chassis_width}"
+    chassis_height="${chassis_height}"
+    wheel_mass="${wheel_mass}"
+    wheel_radius="${wheel_radius}"
+    wheel_width="${wheel_width}"
+    wheel_base="${wheel_base}"
+    wheel_track="${wheel_track}"
+    steering_mass="${steering_mass}"
+    steering_radius="${steering_radius}"
+    steering_thickness="${steering_thickness}"
+    offset="${wheel_offset}"
+    x_reflect="${front_x_reflect}"
+    y_reflect="${right_y_reflect}"
+    steer_joint_damping="0.05" steer_joint_friction="0.0"
+    wheel_joint_damping="0.02" wheel_joint_friction="0.0"/>
+  <xacro:drive_module_assembly
+    name="left_rear"
+    chassis_length="${chassis_length}"
+    chassis_width="${chassis_width}"
+    chassis_height="${chassis_height}"
+    wheel_mass="${wheel_mass}"
+    wheel_radius="${wheel_radius}"
+    wheel_width="${wheel_width}"
+    wheel_base="${wheel_base}"
+    wheel_track="${wheel_track}"
+    steering_mass="${steering_mass}"
+    steering_radius="${steering_radius}"
+    steering_thickness="${steering_thickness}"
+    offset="${wheel_offset}"
+    x_reflect="${rear_x_reflect}"
+    y_reflect="${left_y_reflect}"
+    steer_joint_damping="0.05" steer_joint_friction="0.0"
+    wheel_joint_damping="0.02" wheel_joint_friction="0.0"/>
+  <xacro:caster_module_assembly
+    name="left_front"
+    chassis_length="${chassis_length}"
+    chassis_width="${chassis_width}"
+    chassis_height="${chassis_height}"
+    wheel_mass="${wheel_mass}"
+    wheel_radius="${wheel_radius}"
+    wheel_width="${wheel_width}"
+    wheel_base="${wheel_base}"
+    wheel_track="${wheel_track}"
+    steering_mass="${steering_mass}"
+    steering_radius="${steering_radius}"
+    steering_thickness="${steering_thickness}"
+    offset="${wheel_offset}"
+    x_reflect="${front_x_reflect}"
+    y_reflect="${left_y_reflect}"
+    caster_trail="${caster_trail}"
+    steer_joint_damping="0.02" steer_joint_friction="0.0"
+    wheel_joint_damping="0.01" wheel_joint_friction="0.0"/>
+  <xacro:caster_module_assembly
+    name="right_rear"
+    chassis_length="${chassis_length}"
+    chassis_width="${chassis_width}"
+    chassis_height="${chassis_height}"
+    wheel_mass="${wheel_mass}"
+    wheel_radius="${wheel_radius}"
+    wheel_width="${wheel_width}"
+    wheel_base="${wheel_base}"
+    wheel_track="${wheel_track}"
+    steering_mass="${steering_mass}"
+    steering_radius="${steering_radius}"
+    steering_thickness="${steering_thickness}"
+    offset="${wheel_offset}"
+    x_reflect="${rear_x_reflect}"
+    y_reflect="${right_y_reflect}"
+    caster_trail="${caster_trail}"
+    steer_joint_damping="0.02" steer_joint_friction="0.0"
+    wheel_joint_damping="0.01" wheel_joint_friction="0.0"/>
+  <!-- =========================================================
+       4) ros2_control
+       ========================================================= -->
+  <ros2_control name="HamrJointControl" type="system">
+    <hardware>
+      <plugin>gz_ros2_control/GazeboSimSystem</plugin>
+    </hardware>
+    <!-- 구동 모듈만 컨트롤러에 포함 -->
+    <xacro:steering_module_controller name="right_front"/>
+    <xacro:steering_module_controller name="left_rear"/>
+  </ros2_control>
+  <!-- =========================================================
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