Commit message: update ammr sj xacro

File: description/ammr_sj/ammr_sj_gazebo.xacro (robot description, xacro)
@@ -1,11 +1,4 @@
 <?xml version="1.0" ?>
-<robot name="ammr_sj" xmlns:xacro="http://www.ros.org/wiki/xacro" >
-    <!--
-        GAZEBO MACROS
-    -->
-    <!--
-        Define Gazebo specific macro's here because this file isn't included if we're not running
-        Gazebo
-    -->
+<robot name="zinger" xmlns:xacro="http://www.ros.org/wiki/xacro" >
     <xacro:macro name="gazebo_reference_link_wheel" params="name">
         <gazebo reference="link_wheel_${name}">
@@ -20,72 +13,20 @@
         </gazebo>
     </xacro:macro>
-    <xacro:macro name="gazebo_reference_caster_wheel" params="name">
-        <gazebo reference="link_caster_${name}">
-            <mu1>0.9</mu1>
-            <mu2>0.9</mu2>
-            <kp>500000.0</kp>
-            <kd>10.0</kd>
-            <minDepth>0.001</minDepth>
-            <maxVel>0.1</maxVel>
-            <fdir1>1 0 0</fdir1>
-            <selfCollide>true</selfCollide>
-        </gazebo>
-    </xacro:macro>
     <!-- Sensors -->
-    <xacro:macro name="gazebo_sensor_imu" params="name update_rate:=25" >
-        <gazebo reference="${name}">
+    <xacro:macro name="gazebo_sensor_imu" params="name update_rate:=100">
+        <gazebo reference="link_sensor_imu_${name}">
             <sensor name="${name}" type="imu">
-                <gz_frame_id>${name}</gz_frame_id>
                 <always_on>true</always_on>
                 <update_rate>${update_rate}</update_rate>
-                <imu>
-                    <angular_velocity>
-                    <x>
-                        <noise type="gaussian">
-                        <mean>0.0</mean>
-                        <stddev>0.0</stddev>
-                        </noise>
-                    </x>
-                    <y>
-                        <noise type="gaussian">
-                        <mean>0.0</mean>
-                        <stddev>0.0</stddev>
-                        </noise>
-                    </y>
-                    <z>
-                        <noise type="gaussian">
-                        <mean>0.0</mean>
-                        <stddev>0.0</stddev>
-                        </noise>
-                    </z>
-                    </angular_velocity>
-                    <linear_acceleration>
-                    <x>
-                        <noise type="gaussian">
-                        <mean>0.0</mean>
-                        <stddev>0.0</stddev>
-                        </noise>
-                    </x>
-                    <y>
-                        <noise type="gaussian">
-                        <mean>0.0</mean>
-                        <stddev>0.0</stddev>
-                        </noise>
-                    </y>
-                    <z>
-                        <noise type="gaussian">
-                        <mean>0.0</mean>
-                        <stddev>0.0</stddev>
-                        </noise>
-                    </z>
-                    </linear_acceleration>
-                </imu>
+                <gz_frame_id>link_sensor_imu_${name}</gz_frame_id>
+                <!-- gz transport topic 이름 (ROS2 토픽 아님) -->
+                <topic>imu</topic>
                 <plugin
-                        filename="gz-sim-imu-system"
-                        name="gz::sim::systems::Imu">
+                    filename="gz-sim-imu-system"
+                    name="gz::sim::systems::Imu">
                     <alwaysOn>true</alwaysOn>
-                    <updateRate>25</updateRate>
+                    <updateRate>${update_rate}</updateRate>
                     <topic>imu</topic>
-                    <imuName>imu_center</imuName>
+                    <imuName>${name}</imuName>
                 </plugin>
             </sensor>
@@ -95,62 +36,60 @@
         </gazebo>
     </xacro:macro>
-    <xacro:macro name="gazebo_sensor_lidar" params="name topic_name" >
-        <gazebo reference="${name}">
+    <xacro:macro name="gazebo_sensor_lidar" params="name reference_link topic">
+        <gazebo reference="${reference_link}">
             <sensor name="${name}" type="gpu_lidar">
                 <pose>0 0 0.02 0 0 0</pose>
                 <always_on>true</always_on>
-                <topic>${topic_name}</topic>
-                <update_rate>30</update_rate>
+                <topic>${topic}</topic>
+                <update_rate>20</update_rate>
                 <lidarName>${name}</lidarName>
                 <visualize>true</visualize>
-                <gz_frame_id>${name}</gz_frame_id>
+                <gz_frame_id>${reference_link}</gz_frame_id>
                 <lidar>
                     <scan>
-                        <horizontal>
-                            <samples>640</samples>
-                            <resolution>1.0</resolution>
-                            <min_angle>${-pi}</min_angle>
-                            <max_angle>${pi}</max_angle>
-                        </horizontal>
+                    <horizontal>
+                        <samples>1440</samples>
+                        <resolution>1</resolution>
+                        <min_angle>-2.35619</min_angle>
+                        <max_angle>2.35619</max_angle>
+                    </horizontal>
                     </scan>
                     <range>
-                        <min>0.55</min>
-                        <max>16.0</max>
-                        <resolution>0.01</resolution>
+                    <min>0.05</min>
+                    <max>40.0</max>
+                    <resolution>0.01</resolution>
                     </range>
+                    <noise>
+                    <type>gaussian</type>
+                    <mean>0.0</mean>
+                    <stddev>0.01</stddev>
+                    </noise>
                 </lidar>
-                <plugin
-                    filename="gz-sim-sensors-system"
-                    name="gz::sim::systems::Sensors">
-                    <render_engine>ogre2</render_engine>
-                </plugin>
             </sensor>
         </gazebo>
+        <gazebo reference="joint_body_to_sensor_lidar_${name}">
+            <preserveFixedJoint>true</preserveFixedJoint>
+        </gazebo>
     </xacro:macro>
-    <!--
-        GAZEBO
-    -->
-    <!-- Motorized wheels -->
+    <xacro:gazebo_reference_link_wheel name="left_front" />
+    <xacro:gazebo_reference_link_wheel name="left_rear" />
+    <xacro:gazebo_reference_link_wheel name="right_rear" />
     <xacro:gazebo_reference_link_wheel name="right_front" />
-    <xacro:gazebo_reference_link_wheel name="left_rear" />
-    <!-- Caster wheels -->
-    <xacro:gazebo_reference_caster_wheel name="left_front" />
-    <xacro:gazebo_reference_caster_wheel name="right_rear" />
-    <xacro:gazebo_sensor_imu name="imu_frame" />
-    <xacro:gazebo_sensor_lidar name="lidar_front" topic_name="/scan_front" />
-    <xacro:gazebo_sensor_lidar name="lidar_back" topic_name="/scan_rear" />
+    <xacro:gazebo_sensor_imu name="center" />
+    <xacro:gazebo_sensor_lidar name="lidar_front" reference_link="lidar_front" topic="/scan_front"/>
+    <xacro:gazebo_sensor_lidar name="lidar_back"  reference_link="lidar_back"  topic="/scan_rear"/>
     <gazebo>
+        <plugin filename="gz-sim-sensors-system"
+                name="gz::sim::systems::Sensors">
+            <render_engine>ogre2</render_engine>
+        </plugin>
         <plugin filename="gz-sim-joint-state-publisher-system"
                 name="gz::sim::systems::JointStatePublisher">
         </plugin>
-        <plugin
-                filename="gz_ros2_control-system"
+        <plugin filename="gz_ros2_control-system"
                 name="gz_ros2_control::GazeboSimROS2ControlPlugin">
             <parameters>${param_file}</parameters>
         </plugin>
-    </gazebo>
-    <!-- <gazebo>
-         <plugin
-                filename="gz-sim-pose-publisher-system"
+        <!-- <plugin filename="gz-sim-pose-publisher-system"
                 name="gz::sim::systems::PosePublisher">
             <publish_link_pose>true</publish_link_pose>
@@ -163,5 +102,14 @@
             <static_publisher>true</static_publisher>
             <static_update_frequency>-1</static_update_frequency>
-        </plugin>
-    </gazebo> -->
+        </plugin> -->
+        <!-- <plugin filename="gz-sim-odometry-publisher-system"
+              name="gz::sim::systems::OdometryPublisher">
+            <odom_frame>odom</odom_frame>
+            <robot_base_frame>base_footprint</robot_base_frame>
+            <odom_topic>/odom</odom_topic>
+            <tf_topic>/tf</tf_topic>
+            <dimensions>2</dimensions>
+            <odom_publish_frequency>20</odom_publish_frequency>
+        </plugin> -->
+    </gazebo>
 </robot>

File: description/ammr_sj/ammr_sj_macros.xacro (robot description, xacro)
@@ -1,4 +1,4 @@
 <?xml version="1.0" ?>
-<robot name="ammr_sj" xmlns:xacro="http://www.ros.org/wiki/xacro" >
+<robot name="zinger" xmlns:xacro="http://www.ros.org/wiki/xacro" >
     <!--
         A macro to create a wheel link and the joint for the wheel
@@ -9,11 +9,21 @@
         - width: Width of the wheel in meters
         - offset: The distance between the wheel and the steering plate above the wheel. In meters.
+        [ADDED]
+        - caster_trail: steering 축 기준 wheel을 x(-)로 빼는 값(=트레일). caster 정렬성에 매우 중요
+        - wheel_joint_damping / wheel_joint_friction: wheel spin 조인트 동특성
     -->
-    <xacro:macro name="wheel_assembly" params="name mass radius width offset">
+    <xacro:macro name="wheel_assembly"
+                 params="name mass radius width offset
+                         caster_trail:=0.0
+                         wheel_joint_damping:=0.02
+                         wheel_joint_friction:=0.0">
         <joint name="joint_steering_to_wheel_${name}" type="continuous">
-            <origin rpy="0 0 0" xyz="0 0 ${-1 * (radius + offset -0.005)}"/>
+            <!-- 핵심: caster_trail 적용 -->
+            <origin rpy="0 0 0" xyz="${-caster_trail} 0 ${-1 * (radius + offset)}"/>
             <parent link="link_steering_${name}"/>
             <child link="link_wheel_${name}"/>
             <axis xyz="0.0 1.0 0.0"/>
+            <!-- wheel이 잘 굴러가게 -->
+            <dynamics damping="${wheel_joint_damping}" friction="${wheel_joint_friction}"/>
         </joint>
         <link name="link_wheel_${name}">
@@ -45,47 +55,4 @@
     </xacro:macro>
     <!--
-        A macro to create a caster wheel (passive wheel)
-        Parameters:
-        - name: Name of the caster, e.g. left_front
-        - mass: Mass of the caster wheel in kilogram
-        - radius: Radius of the caster wheel in meters
-        - width: Width of the caster wheel in meters
-        - x_pos: X position relative to base_link center
-        - y_pos: Y position relative to base_link center
-    -->
-    <xacro:macro name="caster_wheel_assembly" params="name mass radius width x_pos y_pos">
-        <joint name="joint_chassis_to_caster_${name}" type="fixed">
-            <parent link="base_link"/>
-            <child link="link_caster_${name}"/>
-            <origin rpy="0 0 0" xyz="${x_pos} ${y_pos} ${radius}"/>
-        </joint>
-        <link name="link_caster_${name}">
-            <inertial>
-                <origin xyz="0 0 0" rpy="${PI/2} 0 0" />
-                <mass value="${mass}"/>
-                <inertia
-                    ixx="${(mass/12) * (3*radius*radius + width*width)}"
-                    ixy="0"
-                    ixz="0"
-                    iyy="${(mass/12) * (3*radius*radius + width*width)}"
-                    iyz="0"
-                    izz="${(mass/2) * (radius*radius)}"/>
-            </inertial>
-            <visual>
-                <origin rpy="${PI/2} 0 0" xyz="0 0 0"/>
-                <geometry>
-                    <cylinder length="${width}" radius="${radius}" />
-                </geometry>
-                <material name="gray"/>
-            </visual>
-            <collision>
-                <origin rpy="${PI/2} 0 0" xyz="0 0 0"/>
-                <geometry>
-                    <cylinder length="${width}" radius="${radius}" />
-                </geometry>
-            </collision>
-        </link>
-    </xacro:macro>
-    <!--
         A macro to create a steering link and the joint for the steering unit
         Parameters:
@@ -97,15 +64,29 @@
         - steering_radius: Radius of the steering unit in meters
         - wheel_radius: Radius of the wheel in meters
+        - wheel_base: Base of the wheel in meters
+        - wheel_track: Track of the wheel in meters
         - thickness: Thickness of the steering unit
         - offset: The distance between the wheel and the steering plate above the wheel. In meters.
         - x_reflect: Direction multiplier for X offsets. Either 1 or -1
         - y_reflect: Direction multiplier for Y offsets. Either 1 or -1
+        [ADDED]
+        - steer_joint_damping / steer_joint_friction: steering yaw 조인트 동특성
     -->
-    <xacro:macro name="steering_assembly" params="name mass chassis_length chassis_width chassis_height steering_radius thickness wheel_radius wheel_base wheel_track offset x_reflect y_reflect">
+    <xacro:macro name="steering_assembly"
+                 params="name mass chassis_length chassis_width chassis_height
+                         steering_radius thickness wheel_radius wheel_base wheel_track offset
+                         x_reflect y_reflect
+                         steer_joint_damping:=0.05
+                         steer_joint_friction:=0.0">
         <joint name="joint_chassis_to_steering_${name}" type="continuous">
-            <origin rpy="0 0 0" xyz="${x_reflect * (0.5 * wheel_base)} ${y_reflect * (0.5 * wheel_track)} ${wheel_radius + offset}"/>
-            <parent link="base_link"/>
+            <origin rpy="0 0 0"
+                    xyz="${x_reflect * (0.5 * wheel_base)}
+                        ${y_reflect * (0.5 * wheel_track)}
+                        ${-(0.5 * chassis_height + chassis_bottom_z) + (2 * wheel_radius) + offset + (0.5 * thickness)}"/>
+            <parent link="chassis_link"/>
             <child link="link_steering_${name}"/>
             <axis xyz="0.0 0.0 1.0"/>
+            <!-- steering이 쉽게 돌아가게 -->
+            <dynamics damping="${steer_joint_damping}" friction="${steer_joint_friction}"/>
         </joint>
         <link name="link_steering_${name}">
@@ -150,5 +131,5 @@
     </xacro:macro>
     <!--
-        A macro to create a wheel link and the joint for the wheel
+        A macro to create a drive module (steering + wheel) for powered swerve
         Parameters:
         - name: Name of the wheel, e.g. left_rear
@@ -162,6 +143,15 @@
         - x_reflect: Direction multiplier for X offsets. Either 1 or -1
         - y_reflect: Direction multiplier for Y offsets. Either 1 or -1
+        [ADDED: pass-through defaults for dynamics + caster_trail]
+        - caster_trail: 기본은 0 (구동 모듈은 굳이 캐스터 트레일 필요 없음)
     -->
-    <xacro:macro name="drive_module_assembly" params="name chassis_length chassis_width chassis_height wheel_mass wheel_radius wheel_width wheel_base wheel_track steering_mass steering_radius steering_thickness offset x_reflect y_reflect">
+    <xacro:macro name="drive_module_assembly"
+                 params="name chassis_length chassis_width chassis_height
+                         wheel_mass wheel_radius wheel_width wheel_base wheel_track
+                         steering_mass steering_radius steering_thickness
+                         offset x_reflect y_reflect
+                         caster_trail:=0.0
+                         steer_joint_damping:=0.05 steer_joint_friction:=0.0
+                         wheel_joint_damping:=0.02 wheel_joint_friction:=0.0">
         <xacro:steering_assembly
             name="${name}"
@@ -177,5 +167,7 @@
             offset="${offset}"
             x_reflect="${x_reflect}"
-            y_reflect="${y_reflect}"/>
+            y_reflect="${y_reflect}"
+            steer_joint_damping="${steer_joint_damping}"
+            steer_joint_friction="${steer_joint_friction}"/>
         <xacro:wheel_assembly
             name="${name}"
@@ -183,5 +175,47 @@
             radius="${wheel_radius}"
             width="${wheel_width}"
-            offset="${offset + 0.5 * steering_thickness}"/>
+            offset="${offset + 0.5 * steering_thickness}"
+            caster_trail="${caster_trail}"
+            wheel_joint_damping="${wheel_joint_damping}"
+            wheel_joint_friction="${wheel_joint_friction}"/>
+    </xacro:macro>
+    <!--
+        A macro to create an unpowered caster module (steering + wheel)
+        - drive_module_assembly와 동일 구조지만, hamr에서 컨트롤러에 포함시키지 않으면 캐스터로 동작
+        [ADDED]
+    -->
+    <xacro:macro name="caster_module_assembly"
+                 params="name chassis_length chassis_width chassis_height
+                         wheel_mass wheel_radius wheel_width wheel_base wheel_track
+                         steering_mass steering_radius steering_thickness
+                         offset x_reflect y_reflect
+                         caster_trail:=0.01
+                         steer_joint_damping:=0.02 steer_joint_friction:=0.0
+                         wheel_joint_damping:=0.01 wheel_joint_friction:=0.0">
+        <xacro:steering_assembly
+            name="${name}"
+            mass="${steering_mass}"
+            chassis_length="${chassis_length}"
+            chassis_width="${chassis_width}"
+            chassis_height="${chassis_height}"
+            wheel_base="${wheel_base}"
+            wheel_track="${wheel_track}"
+            steering_radius="${steering_radius}"
+            thickness="${steering_thickness}"
+            wheel_radius="${wheel_radius}"
+            offset="${offset}"
+            x_reflect="${x_reflect}"
+            y_reflect="${y_reflect}"
+            steer_joint_damping="${steer_joint_damping}"
+            steer_joint_friction="${steer_joint_friction}"/>
+        <xacro:wheel_assembly
+            name="${name}"
+            mass="${wheel_mass}"
+            radius="${wheel_radius}"
+            width="${wheel_width}"
+            offset="${offset + 0.5 * steering_thickness}"
+            caster_trail="${caster_trail}"
+            wheel_joint_damping="${wheel_joint_damping}"
+            wheel_joint_friction="${wheel_joint_friction}"/>
     </xacro:macro>
     <!-- CONTROLLERS -->
@@ -208,5 +242,5 @@
     <!-- SENSORS -->
     <!-- IMU sensor -->
-    <xacro:macro name="imu_frame" params="name parent_link *origin">
+    <xacro:macro name="sensor_imu" params="name parent_link *origin">
         <xacro:property name="mass"     value="0.01"/>
         <xacro:property name="length_x" value="0.01" />
@@ -217,9 +251,9 @@
         <xacro:property name="collision_z_offset" value="${0.5 * length_z}" />
         <joint name="joint_body_to_sensor_imu_${name}" type="fixed">
+            <xacro:insert_block name="origin"/>
             <parent link="${parent_link}"/>
-            <child link="${name}"/>
-            <origin xyz="0.0 0.0 0.0"/>
-        </joint>
-        <link name="${name}">
+            <child link="link_sensor_imu_${name}"/>
+        </joint>
+        <link name="link_sensor_imu_${name}">
             <visual>
                 <origin xyz="${collision_x_offset} ${collision_y_offset} ${collision_z_offset}"/>
@@ -247,21 +281,21 @@
         </link>
     </xacro:macro>
-    <!-- Base_scan == Lidar Center  sensor -->
-    <xacro:macro name="sensor_lidar" params="name parent_link chassis_top_relative_height">
-        <xacro:property name="mass"     value="0.17"/>
-        <xacro:property name="length_x" value="0.071" />
-        <xacro:property name="length_y" value="0.10" />
-        <xacro:property name="length_z" value="0.06" />
+    <!-- Lidar sensor -->
+    <xacro:macro name="sensor_lidar" params="name parent_link *origin">
+        <xacro:property name="mass"     value="1.0"/>
+        <xacro:property name="length_x" value="0.15" />
+        <xacro:property name="length_y" value="0.15" />
+        <xacro:property name="length_z" value="0.15" />
         <xacro:property name="collision_x_offset" value="0" />
         <xacro:property name="collision_y_offset" value="0" />
-        <xacro:property name="collision_z_offset" value="${chassis_top_relative_height}" />
+        <xacro:property name="collision_z_offset" value="0" />
         <joint name="joint_body_to_sensor_lidar_${name}" type="fixed">
+            <xacro:insert_block name="origin"/>
             <parent link="${parent_link}"/>
             <child link="link_sensor_lidar_${name}"/>
-            <origin rpy="0 0 0" xyz="${collision_x_offset} ${collision_y_offset} ${collision_z_offset}"/>
         </joint>
         <link name="link_sensor_lidar_${name}">
             <visual>
-                <origin rpy="0 0 0" xyz="0.0 0 ${0.5 * length_z}"/>
+                <origin rpy="0.0 0.0 0.0" xyz="0.0 0.0 0.0"/>
                 <geometry>
                     <box size="${length_x} ${length_y} ${length_z}"/>
@@ -269,5 +303,5 @@
             </visual>
             <collision>
-                <origin rpy="0 0 0" xyz="0.0 0 ${0.5 * length_z}"/>
+                <origin rpy="0.0 0.0 0.0" xyz="0.0 0.0 0.0"/>
                 <geometry>
                     <box size="${length_x} ${length_y} ${length_z}"/>
@@ -276,5 +310,5 @@
             <inertial>
                 <mass value="${mass}" />
-                <origin rpy="0 0 0" xyz="0.0 0 ${0.5 * length_z}"/>
+                <origin rpy="0.0 0.0 0.0" xyz="0.0 0.0 0.0"/>
                 <inertia
                     ixx="${(1/12) * mass * (length_y*length_y + length_z*length_z)}"
@@ -287,6 +321,3 @@
         </link>
     </xacro:macro>
-    <!-- Bump sensor -->
-    <!-- Sonar sensor -->
-    <!-- IR sensor -->
 </robot>

Commit message: fix wheel radius

File: description/ammr_sj/ammr_sj.xacro (robot description, xacro)
@@ -24,5 +24,5 @@
   <!-- Wheel dimensions -->
   <xacro:property name="wheel_mass" value="0.2"/>
-  <xacro:property name="wheel_radius" value="0.15"/>
+  <xacro:property name="wheel_radius" value="0.075"/>
   <xacro:property name="wheel_width" value="0.04"/>
   <xacro:property name="wheel_base" value="0.728"/>
