Commit message: add p2bot hload

File: description/p2bot_hload/p2bot_hload.xacro (robot description, xacro)
@@ -1,36 +1,45 @@
 <?xml version="1.0"?>
 <!--
-  p2bot — STMF P2 differential-drive robot (Gazebo sanity 데모, §2.7). namespace-aware.
-  bcr_bot의 '형태'(diff 구동계·센서 구성)만 참고, 외형 mesh 없음(저널 사진용 primitive).
-  치수: 폭 0.6 · 길이 0.7 · 높이 ~0.35 m (1.0m 지름길을 여유있게 통과하도록 lift_l 0.8×1.0에서 축소).
-  멀티로봇: namespace 인자 → **링크명·tf frame·topic을 <ns>/ 로 프리픽스**(RViz RobotModel이 tf에
-  붙으려면 URDF 링크명 == tf 프레임명이어야 하므로 링크명 자체를 프리픽스; rsp frame_prefix는 안 씀).
-  단일로봇(namespace=''): base_footprint·/cmd_vel 그대로. joint 이름은 모델 스코프라 프리픽스 안 함.
+  p2bot_hload — STMF P2 H_load (§4.4 정적 제약 대표종). p2bot 구조 그대로, 치수만 [표1] 정합.
+  [표1] H_load: W 1.2 × L 1.5 × H 1.2 m, payload 2000 kg, MANUAL_LOAD
+    - 폭 1.2 > 지름길 통행폭 1.0  -> 빈 상태에서도 두 지름길 모두 차단
+    - 높이 1.2 > aisle_short_1 통행고 1.0 -> 중복 차단
+    => 적재 여부와 무관하게 메인 통로(폭 2.0)만 사용. §4.4의 "왕복 대칭" 대조군.
+  ★ 라이다 z = 0.20 (p2bot은 섀시 상단). 이유: LIFT_M 전고가 0.30 m라
+    섀시 위(≈1.3 m)에 두면 LIFT_M을 아예 감지하지 못한다. 0.20이면
+    H_load 섀시(0.15~1.20)와 LIFT_M 섀시(0.10~0.30)를 서로 잡는다.
+    적재물은 실제로 올리지 않으므로 라이다를 낮춰도 잃는 정보가 없다.
+    섀시 내부 높이라 전방으로 돌출 마운트 -> 후방 사각 발생(주석 참조).
+  ★ 코너 통과가 최대 리스크: 제자리 회전 스윕 반경 sqrt(0.75^2+0.60^2)=0.96 m,
+    지름 1.92 m. corridor_main <-> corridor_load 코너는 2x2 m -> 사방 여유 0.04 m.
+    inflation_radius를 키우면 계획 자체가 안 난다. 실행 전 확인 1순위.
 -->
-<robot xmlns:xacro="http://www.ros.org/wiki/xacro" name="p2bot">
+<robot xmlns:xacro="http://www.ros.org/wiki/xacro" name="p2bot_hload">
   <!-- ..................... namespace / prefix ..................... -->
   <xacro:arg name="namespace" default=""/>
   <xacro:property name="ns" value="$(arg namespace)"/>
-  <xacro:property name="fp" value="${ns + '/' if ns != '' else ''}"/>   <!-- link/frame/topic prefix -->
-  <!-- ..................... 치수 (지름길 통과용 축소) ..................... -->
-  <xacro:property name="chassis_l" value="0.7"/>
-  <xacro:property name="chassis_w" value="0.6"/>
-  <xacro:property name="chassis_h" value="0.35"/>
-  <xacro:property name="chassis_mass" value="60"/>
-  <xacro:property name="wheel_radius" value="0.10"/>
-  <xacro:property name="wheel_width"  value="0.05"/>
-  <xacro:property name="wheel_track"  value="0.5"/>
-  <xacro:property name="wheel_mass"   value="1.0"/>
-  <xacro:property name="caster_radius" value="0.06"/>
-  <xacro:property name="caster_x" value="0.26"/>
-  <!-- 라이다: H_load와 공통 스캔 평면 z=0.20. 섀시(0.10~0.45) 내부 높이라 전방 돌출 마운트 -->
+  <xacro:property name="fp" value="${ns + '/' if ns != '' else ''}"/>
+  <!-- ..................... 치수 ([표1] H_load) ..................... -->
+  <xacro:property name="chassis_l" value="1.5"/>    <!-- L (x) -->
+  <xacro:property name="chassis_w" value="1.2"/>    <!-- W (y) -->
+  <xacro:property name="total_h"   value="0.8"/>    <!-- 지면~상단 전고 -->
+  <xacro:property name="chassis_mass" value="300"/>
+  <xacro:property name="wheel_radius" value="0.15"/>
+  <xacro:property name="wheel_width"  value="0.10"/>
+  <xacro:property name="wheel_track"  value="1.00"/>
+  <xacro:property name="wheel_mass"   value="8.0"/>
+  <!-- 섀시 박스 높이 = 전고 - 지상고(=바퀴 반경). 섀시 범위 z: 0.15 ~ 1.20 -->
+  <xacro:property name="chassis_h" value="${total_h - wheel_radius}"/>
+  <xacro:property name="caster_radius" value="0.10"/>
+  <xacro:property name="caster_x" value="0.60"/>
+  <!-- 라이다: 월드 z 목표. 섀시 내부 높이이므로 전방 돌출 마운트 -->
   <xacro:property name="lidar_z"      value="0.20"/>
   <xacro:property name="lidar_radius" value="0.05"/>
   <xacro:property name="lidar_x"      value="${chassis_l/2 + lidar_radius}"/>
   <xacro:arg name="two_d_lidar_enabled" default="true"/>
-  <!-- ..................... 재질 (커스텀 색) ..................... -->
-  <material name="p2_body">  <color rgba="0.18 0.45 0.55 1.0"/></material>
-  <material name="p2_wheel"> <color rgba="0.12 0.12 0.13 1.0"/></material>
-  <material name="p2_trim">  <color rgba="0.85 0.85 0.88 1.0"/></material>
+  <!-- ..................... 재질 (H_load 구분색: 진한 주황) ..................... -->
+  <material name="p2_hload_body"> <color rgba="0.72 0.36 0.12 1.0"/></material>
+  <material name="p2_wheel">      <color rgba="0.12 0.12 0.13 1.0"/></material>
+  <material name="p2_trim">       <color rgba="0.85 0.85 0.88 1.0"/></material>
   <!-- ..................... 관성 매크로 ..................... -->
   <xacro:macro name="box_inertia" params="m x y z">
@@ -52,6 +61,5 @@
     </inertial>
   </xacro:macro>
-  <!-- ..................... GAZEBO 플러그인 (모델 레벨만; ns 프리픽스) ..................... -->
-  <!-- sensors/imu 시스템은 서버 레벨(시뮬당 1개)이라 월드(p2.sdf)에 둠 — 멀티로봇 씬 중복 crash 방지. -->
+  <!-- ..................... GAZEBO 플러그인 ..................... -->
   <gazebo>
     <plugin filename="gz-sim-joint-state-publisher-system"
@@ -70,6 +78,14 @@
       <frame_id>${fp}odom</frame_id>
       <child_frame_id>${fp}base_footprint</child_frame_id>
+      <!-- §4.1 시간 모델 v = 1.0 m/s와 정합. 중량체라 가감속·선회는 보수적으로 -->
+      <max_linear_velocity>1.0</max_linear_velocity>
+      <min_linear_velocity>-0.3</min_linear_velocity>
+      <max_angular_velocity>0.5</max_angular_velocity>
+      <min_angular_velocity>-0.5</min_angular_velocity>
+      <max_linear_acceleration>0.4</max_linear_acceleration>
+      <min_linear_acceleration>-0.4</min_linear_acceleration>
+      <max_angular_acceleration>0.8</max_angular_acceleration>
+      <min_angular_acceleration>-0.8</min_angular_acceleration>
     </plugin>
-    <!-- ground-truth odom + tf(odom→base_footprint). tf는 로봇별 gz토픽 /{ns}/tf -->
     <plugin filename="gz-sim-odometry-publisher-system"
             name="gz::sim::systems::OdometryPublisher">
@@ -82,5 +98,5 @@
     </plugin>
   </gazebo>
-  <!-- ..................... BASE (링크명 프리픽스) ..................... -->
+  <!-- ..................... BASE ..................... -->
   <link name="${fp}base_footprint"/>
   <link name="${fp}base_link"/>
@@ -94,5 +110,5 @@
     <visual>
       <geometry><box size="${chassis_l} ${chassis_w} ${chassis_h}"/></geometry>
-      <material name="p2_body"/>
+      <material name="p2_hload_body"/>
     </visual>
     <xacro:box_inertia m="${chassis_mass}" x="${chassis_l}" y="${chassis_w}" z="${chassis_h}"/>
@@ -102,6 +118,6 @@
     <origin xyz="0 0 0" rpy="0 0 0"/>
   </joint>
-  <gazebo reference="${fp}chassis_link"><material>Gazebo/Turquoise</material></gazebo>
-  <!-- ..................... 구동륜 (joint 이름은 프리픽스 안 함, 링크는 함) ..................... -->
+  <gazebo reference="${fp}chassis_link"><material>Gazebo/Orange</material></gazebo>
+  <!-- ..................... 구동륜 ..................... -->
   <xacro:macro name="drive_wheel" params="side reflect">
     <link name="${fp}${side}_wheel">
@@ -130,5 +146,5 @@
   <xacro:drive_wheel side="left"  reflect="1"/>
   <xacro:drive_wheel side="right" reflect="-1"/>
-  <!-- ..................... 캐스터 ..................... -->
+  <!-- ..................... 캐스터 (전후 각 1, 장축 1.5 m 지지) ..................... -->
   <xacro:macro name="caster" params="side sign">
     <link name="${fp}caster_${side}">
@@ -138,5 +154,5 @@
       </collision>
       <visual><geometry><sphere radius="${caster_radius}"/></geometry><material name="p2_trim"/></visual>
-      <xacro:sph_inertia m="0.1" r="${caster_radius}"/>
+      <xacro:sph_inertia m="2.0" r="${caster_radius}"/>
     </link>
     <joint name="caster_${side}_joint" type="fixed">
@@ -148,5 +164,11 @@
   <xacro:caster side="front" sign="1"/>
   <xacro:caster side="back"  sign="-1"/>
-  <!-- ..................... 2D LIDAR (/{ns}/scan) ..................... -->
+  <!-- ..................... 2D LIDAR — 저위치 전방 돌출 ..................... -->
+  <!--
+    z=0.20: LIFT_M(전고 0.30)을 감지하기 위한 필수 조건. 섀시 위면 못 본다.
+    x=+0.80: 섀시(전면 0.75) 밖으로 빼야 시야가 열린다. collision 없음(footprint 불변).
+    후방 사각: 마주 오는 상황은 양쪽이 서로를 보고, 뒤에서 접근하는 쪽은
+      그쪽 로봇이 회피하므로 우선 전방 단독. 부족하면 대각 2개(전좌/후우)로 확장.
+  -->
   <xacro:if value="$(arg two_d_lidar_enabled)">
     <link name="${fp}two_d_lidar">
@@ -167,5 +189,5 @@
           <scan><horizontal>
             <samples>1500</samples><resolution>1</resolution>
-            <min_angle>${radians(-89)}</min_angle><max_angle>${radians(89)}</max_angle>
+            <min_angle>${radians(-94)}</min_angle><max_angle>${radians(94)}</max_angle>
           </horizontal></scan>
           <range><min>0.05</min><max>40.0</max><resolution>0.01</resolution></range>
