Commit message: fix lidar position and nav param

File: description/p2bot_lift_l/p2bot_lift_l.xacro (robot description, xacro)
@@ -39,5 +39,5 @@
   <xacro:property name="lidar_z"      value="0.2"/>
   <xacro:property name="lidar_radius" value="0.05"/>
-  <xacro:property name="lidar_x"      value="${chassis_l/2 + lidar_radius}"/>
+  <xacro:property name="lidar_x" value="${chassis_l/2}"/>
   <xacro:arg name="two_d_lidar_enabled" default="true"/>
   <!-- ..................... 재질 ..................... -->

File: description/p2bot_lift_m/p2bot_lift_m.xacro (robot description, xacro)
@@ -45,5 +45,5 @@
   <xacro:property name="lidar_z"      value="0.20"/>
   <xacro:property name="lidar_radius" value="0.05"/>
-  <xacro:property name="lidar_x"      value="${chassis_l/2 + lidar_radius}"/>
+  <xacro:property name="lidar_x" value="${chassis_l/2}"/>
   <xacro:arg name="two_d_lidar_enabled" default="true"/>
   <!-- ..................... 재질 (커스텀 색) ..................... -->
